Commit message: feat(costmap): finish uint8 cost-field refactor + close avoidance loop
Finish bool->uint8 cost-field refactor (NAV2-aligned) and fix the avoidance loop so the SceneSimulator demo drives (2,0) around box(8,0) to goal (15,0).

- OccupancyGrid cells bool->uint8 (FREE/INSCRIBED/LETHAL + exp inflation)
- A* cost-aware; ScanToGrid /scan raytrace; GridUpdater centroid+inflation
- decision: scan raytrace + objects (chassis->map TF) write the grid
- inscribed_radius 0.22->0.35 (A* no-go zone >= guard stop_dist; path no longer grazes box)
- motor_ctrl guard diagnostic log; VFH off in demo (conflicts with A* in multi-obstacle scene)

Tests 24/24 green. Round-trip patrol left as follow-up (scene latched cmd_vel drift + decision doesn't replan after goal completion).

Co-Authored-By: Claude <noreply@anthropic.com>

File: worlds/amr_visual.urdf (robot description, URDF)
Before this commit: robot amr, 5 links, 4 joints
Links:
- removed link amr/odom
Joints:
- removed joint base_joint
